File: cad/v2.1.0.0/julia_v2.1.0.0/julia_config.sch (KiCad schematic (older format))
At the start: 8 parts, among them U5 W25Q80DVSNIG, U6 EFM8BB21F16I-C-QFN20

Commit message: v2.1.0.0: changed connector, ERC, annotation/footprint assignment
Parts:
- C41: footprint (none) -> Capacitor_SMD:C_0603_1608Metric
- C42: footprint (none) -> Capacitor_SMD:C_0402_1005Metric
- R5, R6, R7, R8: footprint (none) -> Resistor_SMD:R_0402_1005Metric
Changed lines of the file:
@@
 $Descr A4 11693 8268
 encoding utf-8
-Sheet 6 7
+Sheet 4 7
 Title ""
 Date ""
@@
 F 0 "R5" H 3220 1796 50  0000 L CNN
 F 1 "10k" H 3220 1705 50  0000 L CNN
-F 2 "" V 3080 1750 50  0001 C CNN
+F 2 "Resistor_SMD:R_0402_1005Metric" V 3080 1750 50  0001 C CNN
 F 3 "~" H 3150 1750 50  0001 C CNN
 	1    3150 1750
@@
 F 0 "C41" H 2415 1796 50  0000 L CNN
 F 1 "1uF" H 2415 1705 50  0000 L CNN
-F 2 "" H 2338 1600 50  0001 C CNN
+F 2 "Capacitor_SMD:C_0603_1608Metric" H 2338 1600 50  0001 C CNN
 F 3 "~" H 2300 1750 50  0001 C CNN
 	1    2300 1750
@@
 F 0 "C42" H 2765 1796 50  0000 L CNN
 F 1 "0.1uF" H 2765 1705 50  0000 L CNN
-F 2 "" H 2688 1600 50  0001 C CNN
+F 2 "Capacitor_SMD:C_0402_1005Metric" H 2688 1600 50  0001 C CNN
 F 3 "~" H 2650 1750 50  0001 C CNN
 	1    2650 1750
@@
 F 0 "R6" H 3520 4846 50  0000 L CNN
 F 1 "10k" H 3520 4755 50  0000 L CNN
-F 2 "" V 3380 4800 50  0001 C CNN
+F 2 "Resistor_SMD:R_0402_1005Metric" V 3380 4800 50  0001 C CNN
 F 3 "~" H 3450 4800 50  0001 C CNN
 	1    3450 4800
@@
 F 0 "R7" H 5920 4846 50  0000 L CNN
 F 1 "10k" H 5920 4755 50  0000 L CNN
-F 2 "" V 5780 4800 50  0001 C CNN
+F 2 "Resistor_SMD:R_0402_1005Metric" V 5780 4800 50  0001 C CNN
 F 3 "~" H 5850 4800 50  0001 C CNN
 	1    5850 4800
@@
 F 0 "R8" H 6270 4846 50  0000 L CNN
 F 1 "10k" H 6270 4755 50  0000 L CNN
-F 2 "" V 6130 4800 50  0001 C CNN
+F 2 "Resistor_SMD:R_0402_1005Metric" V 6130 4800 50  0001 C CNN
 F 3 "~" H 6200 4800 50  0001 C CNN
 	1    6200 4800
