File: cad/v2.1.0.0/julia_v2.1.0.0/julia_io.sch (KiCad schematic (older format))
At the start: 10 parts, among them J2 JTAG Header, J3 MCU Debug Interface / UART

Commit message: v2.1.0.0: changed connector, ERC, annotation/footprint assignment
Parts:
- removed J3: MCU Debug Interface / UART, symbol Connector_Generic:Conn_02x03_Odd_Even
- D1, D2, D3, D4: footprint (none) -> LED_SMD:LED_0603_1608Metric
- J2: value JTAG Header -> JTAG/C2/UART Header; footprint (none) -> ik:Hirose_DF23_DF23C-10DP-0.5V_2x05_P0.50mm_Vertical
- R1, R2, R3, R4: footprint (none) -> Resistor_SMD:R_0402_1005Metric
Connections:
- wire segments 34 -> 28
- no-connect marks 3 -> 0
Other:
- note removed: "Key on odd side"
Changed lines of the file:
@@
 Text HLabel 1150 1200 0    50   Output ~ 0
 TDI
-Text HLabel 1150 1000 0    50   Output ~ 0
+Text HLabel 1150 1100 0    50   Output ~ 0
 TMS
-Text HLabel 1150 800  0    50   Output ~ 0
+Text HLabel 1150 900  0    50   Output ~ 0
 TCK
-Text HLabel 1150 900  0    50   Input ~ 0
+Text HLabel 1150 1000 0    50   Input ~ 0
 TDO
-$Comp
-L Connector_Generic:Conn_02x05_Odd_Even J2
-U 1 1 605143A5
-P 1650 1000
-F 0 "J2" H 1700 1417 50  0000 C CNN
-F 1 "JTAG Header" H 1700 1326 50  0000 C CNN
-F 2 "" H 1650 1000 50  0001 C CNN
-F 3 "~" H 1650 1000 50  0001 C CNN
-	1    1650 1000
-	1    0    0    -1
-$EndComp
 $Comp
 L power:+3V3 #PWR0125
 U 1 1 60515CBE
-P 2150 700
-F 0 "#PWR0125" H 2150 550 50  0001 C CNN
-F 1 "+3V3" H 2165 873 50  0000 C CNN
-F 2 "" H 2150 700 50  0001 C CNN
-F 3 "" H 2150 700 50  0001 C CNN
-	1    2150 700
+P 1200 700
+F 0 "#PWR0125" H 1200 550 50  0001 C CNN
+F 1 "+3V3" H 1215 873 50  0000 C CNN
+F 2 "" H 1200 700 50  0001 C CNN
+F 3 "" H 1200 700 50  0001 C CNN
+	1    1200 700
 	1    0    0    -1
 $EndComp
@@
 	1    0    0    -1
 $EndComp
-NoConn ~ 1450 1100
-NoConn ~ 1950 1100
-NoConn ~ 1950 1000
-Wire Wire Line
-	1150 800  1450 800
 Wire Wire Line
 	1150 900  1450 900
@@
 	1150 1000 1450 1000
 Wire Wire Line
+	1150 1100 1450 1100
+Wire Wire Line
 	1150 1200 1450 1200
-Wire Wire Line
-	1950 1200 2100 1200
-Wire Wire Line
-	1950 900  2150 900
-Wire Wire Line
-	2150 700  2150 900
-Wire Wire Line
-	1950 800  2100 800
-Wire Wire Line
-	2100 800  2100 1200
-Wire Wire Line
-	2100 1200 2100 1300
-Connection ~ 2100 1200
-Text Notes 1400 1350 0    50   ~ 0
-Key on odd side
-Text HLabel 2900 1050 0    50   BiDi ~ 0
+Text HLabel 2250 1100 2    50   BiDi ~ 0
 C2D
-Text HLabel 2900 1150 0    50   BiDi ~ 0
+Text HLabel 2250 1000 2    50   BiDi ~ 0
 C2CK
-Text HLabel 4000 950  2    50   Input ~ 0
+Text HLabel 2250 800  2    50   Input ~ 0
 UART0_TX
-Text HLabel 4000 1050 2    50   Output ~ 0
+Text HLabel 2250 900  2    50   Output ~ 0
 UART0_RX
 Text HLabel 1200 3100 0    50   Input ~ 0
 MCU_LED1
-$Comp
-L power:+3V3 #PWR0127
-U 1 1 6077B2CF
-P 2900 700
-F 0 "#PWR0127" H 2900 550 50  0001 C CNN
-F 1 "+3V3" H 2915 873 50  0000 C CNN
-F 2 "" H 2900 700 50  0001 C CNN
-F 3 "" H 2900 700 50  0001 C CNN
-	1    2900 700
-	1    0    0    -1
-$EndComp
-$Comp
-L power:GND #PWR0128
-U 1 1 6077B7DB
-P 3850 1350
-F 0 "#PWR0128" H 3850 1100 50  0001 C CNN
-F 1 "GND" H 3855 1177 50  0000 C CNN
-F 2 "" H 3850 1350 50  0001 C CNN
-F 3 "" H 3850 1350 50  0001 C CNN
-	1    3850 1350
-	1    0    0    -1
-$EndComp
-$Comp
-L Connector_Generic:Conn_02x03_Odd_Even J3
-U 1 1 6077C6A3
-P 3400 1050
-F 0 "J3" H 3450 1367 50  0000 C CNN
-F 1 "MCU Debug Interface / UART" H 3450 1276 50  0000 C CNN
-F 2 "" H 3400 1050 50  0001 C CNN
-F 3 "~" H 3400 1050 50  0001 C CNN
-	1    3400 1050
-	1    0    0    -1
-$EndComp
-Wire Wire Line
-	2900 700  2900 950
-Wire Wire Line
-	2900 950  3200 950
-Wire Wire Line
-	3850 1350 3850 1150
-Wire Wire Line
-	3850 1150 3700 1150
-Wire Wire Line
-	2900 1050 3200 1050
-Wire Wire Line
-	2900 1150 3200 1150
-Wire Wire Line
-	3700 950  4000 950
-Wire Wire Line
-	3700 1050 4000 1050
+Wire Wire Line
+	2250 1100 1950 1100
+Wire Wire Line
+	2250 1000 1950 1000
+Wire Wire Line
+	1950 800  2250 800
+Wire Wire Line
+	1950 900  2250 900
 $Comp
 L Device:R R1
@@
 F 0 "R1" H 1420 2846 50  0000 L CNN
 F 1 "470" H 1420 2755 50  0000 L CNN
-F 2 "" V 1280 2800 50  0001 C CNN
+F 2 "Resistor_SMD:R_0402_1005Metric" V 1280 2800 50  0001 C CNN
 F 3 "~" H 1350 2800 50  0001 C CNN
 	1    1350 2800
@@
 F 0 "D1" V 1389 2232 50  0000 R CNN
 F 1 "green" V 1298 2232 50  0000 R CNN
-F 2 "" H 1350 2350 50  0001 C CNN
+F 2 "LED_SMD:LED_0603_1608Metric" H 1350 2350 50  0001 C CNN
 F 3 "~" H 1350 2350 50  0001 C CNN
 	1    1350 2350
@@
 F 0 "R2" H 2270 2846 50  0000 L CNN
 F 1 "470" H 2270 2755 50  0000 L CNN
-F 2 "" V 2130 2800 50  0001 C CNN
+F 2 "Resistor_SMD:R_0402_1005Metric" V 2130 2800 50  0001 C CNN
 F 3 "~" H 2200 2800 50  0001 C CNN
 	1    2200 2800
@@
 F 0 "D2" V 2239 2232 50  0000 R CNN
 F 1 "red" V 2148 2232 50  0000 R CNN
-F 2 "" H 2200 2350 50  0001 C CNN
+F 2 "LED_SMD:LED_0603_1608Metric" H 2200 2350 50  0001 C CNN
 F 3 "~" H 2200 2350 50  0001 C CNN
 	1    2200 2350
@@
 F 0 "R3" H 3170 2846 50  0000 L CNN
 F 1 "470" H 3170 2755 50  0000 L CNN
-F 2 "" V 3030 2800 50  0001 C CNN
+F 2 "Resistor_SMD:R_0402_1005Metric" V 3030 2800 50  0001 C CNN
 F 3 "~" H 3100 2800 50  0001 C CNN
 	1    3100 2800
@@
 F 0 "D3" V 3139 2232 50  0000 R CNN
 F 1 "green" V 3048 2232 50  0000 R CNN
-F 2 "" H 3100 2350 50  0001 C CNN
+F 2 "LED_SMD:LED_0603_1608Metric" H 3100 2350 50  0001 C CNN
 F 3 "~" H 3100 2350 50  0001 C CNN
 	1    3100 2350
@@
 F 0 "R4" H 3970 2846 50  0000 L CNN
 F 1 "470" H 3970 2755 50  0000 L CNN
-F 2 "" V 3830 2800 50  0001 C CNN
+F 2 "Resistor_SMD:R_0402_1005Metric" V 3830 2800 50  0001 C CNN
 F 3 "~" H 3900 2800 50  0001 C CNN
 	1    3900 2800
@@
 F 0 "D4" V 3939 2232 50  0000 R CNN
 F 1 "red" V 3848 2232 50  0000 R CNN
-F 2 "" H 3900 2350 50  0001 C CNN
+F 2 "LED_SMD:LED_0603_1608Metric" H 3900 2350 50  0001 C CNN
 F 3 "~" H 3900 2350 50  0001 C CNN
 	1    3900 2350
@@
 Wire Wire Line
 	3900 2050 3900 2200
+$Comp
+L Connector_Generic:Conn_02x05_Odd_Even J2
+U 1 1 605143A5
+P 1650 1000
+F 0 "J2" H 1700 1417 50  0000 C CNN
+F 1 "JTAG/C2/UART Header" H 1700 1326 50  0000 C CNN
+F 2 "ik:Hirose_DF23_DF23C-10DP-0.5V_2x05_P0.50mm_Vertical" H 1650 1000 50  0001 C CNN
+F 3 "~" H 1650 1000 50  0001 C CNN
+	1    1650 1000
+	1    0    0    -1
+$EndComp
+Wire Wire Line
+	1950 1200 2100 1200
+Wire Wire Line
+	2100 1200 2100 1300
+Wire Wire Line
+	1450 800  1200 800
+Wire Wire Line
+	1200 800  1200 700
 $EndSCHEMATC
