File: cad/v2.1.0.0/julia_v2.1.0.0/julia_v2.1.0.0.kicad_pcb (KiCad board)
At the start: 4 copper layers, 107 parts, among them J1 Barrel_Jack_Switch, J2 JTAG/C2/UART Header, J4 Molex 0541044031, J5 Molex 0522710679, U1 EP4CE6F17, U2 AZ1117-3.3, U3 AZ1117-2.5, U4 NCP565ST12T3G, U5 W25Q80DVSNIG, U6 EFM8BB21F16I-C-QFN20, U7 TPS61165_WSON, U8 AS4C4M32S-7BCN, X1 50MHz

Commit message: Layout complete(?)
Parts:
- removed C21, C23, C26, C30, C34, C36, C40: 0.1uF, Capacitor_SMD:C_0402_1005Metric
- C10, C11, C12, C13, C14, C15, C16, C17, C18, C2, C22, C24, C25, C27, C28, C29, C3, C31, C32, C33, C35, C37, C38, C39, C4, C5, C6, C7, C8, C9, TP2, TP3, TP4, U2, U3, U4: moved to B.Cu
- moved C32 57.8 mm to (104.2, 104.2), turned to 270 degrees
- moved C16 54.8 mm to (97.5, 105.7)
- moved C24 52.1 mm to (105.4, 106.4)
- moved C29 51.7 mm to (101.3, 111.8)
- moved C3 51.2 mm to (120.7, 105.8)
- moved C4 47.9 mm to (116.1, 105.7)
- moved C2 47.2 mm to (122.8, 113.4), turned to 90 degrees
- moved C38 45.5 mm to (95.8, 114.8), turned to 180 degrees
- moved C18 45.4 mm to (121.3, 108.2), turned to 90 degrees
- moved C11 45.4 mm to (115.9, 112.5)
- moved C35 45.3 mm to (93.3, 103.3), turned to 270 degrees
- moved C37 44.9 mm to (97.3, 111.1)
- moved C27 44.6 mm to (98.9, 113.3), turned to 270 degrees
- moved C28 42.0 mm to (108.5, 102.2), turned to 180 degrees
- moved C9 41.8 mm to (108.3, 108.1)
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Connections:
- U1 pad A11: /JuliaFPGA/VSD -> /JuliaFPGA/DEN
- U1 pad B9: /JuliaFPGA/SCL -> /JuliaFPGA/TOUCH_INTN
- U1 pad C9: /JuliaFPGA/TOUCH_INTN -> /JuliaFPGA/SDA
- U1 pad D11: /JuliaFPGA/DEN -> /JuliaFPGA/VSD
- U1 pad D9: /JuliaFPGA/SDA -> /JuliaFPGA/SCL
Routing:
- net +1V2: track 1.37 -> 68.1 mm, vias 2 -> 3
- net +2V5: track 1.33 -> 51.0 mm, vias 2 -> 3
- net /JuliaLCD/LED-: track 0.00 -> 48.4 mm, vias 0 -> 2
- net GND: track 61.4 -> 109.6 mm, vias 74 -> 115
- net +5V: track 0.00 -> 47.9 mm, vias 0 -> 2
- net /JuliaLCD/LED+: track 0.00 -> 42.3 mm
- net /JuliaFPGA/LIGHT: track 4.41 -> 42.5 mm, vias 1 -> 2
- net /JuliaFPGA/TOUCH_RSTN: track 2.52 -> 39.0 mm, vias 0 -> 2
- net /JuliaFPGA/TOUCH_INTN: track 2.48 -> 38.5 mm, vias 0 -> 2
- net /JuliaFPGA/SDA: track 2.52 -> 37.5 mm, vias 0 -> 2
- net /JuliaFPGA/SCL: track 2.56 -> 37.3 mm, vias 0 -> 2
- net +3V3: track 54.9 -> 87.8 mm, vias 63 -> 64
- net /JuliaFPGA/VSD: track 1.30 -> 15.2 mm
- net /JuliaFPGA/HSD: track 0.00 -> 13.1 mm
- net /JuliaFPGA/DEN: track 0.00 -> 12.3 mm
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- added copper zone on B.Cu, net GND
- added copper zone on F.Cu, net GND

Commit message: v2.1.0.0 gerber files
Other:
- board outline added: 60.5 x 46 mm
- board text added: "iank@iank.org v2.1.0.0"
Changed lines of the file:
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@@
   (general
     (thickness 1.6)
-    (drawings 0)
+    (drawings 5)
     (tracks 1806)
     (zones 0)
@@
     (2 In2.Cu power)
     (31 B.Cu signal)
-    (32 B.Adhes user)
-    (33 F.Adhes user)
+    (32 B.Adhes user hide)
+    (33 F.Adhes user hide)
     (34 B.Paste user)
     (35 F.Paste user)
@@
     (43 Eco2.User user hide)
     (44 Edge.Cuts user)
-    (45 Margin user)
-    (46 B.CrtYd user)
-    (47 F.CrtYd user)
+    (45 Margin user hide)
+    (46 B.CrtYd user hide)
+    (47 F.CrtYd user hide)
     (48 B.Fab user hide)
     (49 F.Fab user hide)
@@
     (pad_to_mask_clearance 0)
     (aux_axis_origin 0 0)
-    (grid_origin 68.9 132.8)
+    (grid_origin 78.4 132.8)
     (visible_elements FFFFFF7F)
     (pcbplotparams
@@
       (viasonmask false)
       (mode 1)
-      (useauxorigin false)
+      (useauxorigin true)
       (hpglpennumber 1)
       (hpglpenspeed 20)
@@
       (outputformat 1)
       (mirror false)
-      (drillshape 1)
+      (drillshape 0)
       (scaleselection 1)
-      (outputdirectory ""))
+      (outputdirectory "../../../cam/v2.1.0.0/"))
   )
   (net 0 "")
@@
     (fp_line (start 1.68 -0.95) (end 1.68 0.95) (layer F.CrtYd) (width 0.05))
     (fp_line (start 1.68 0.95) (end -1.68 0.95) (layer F.CrtYd) (width 0.05))
-    (pad 2 smd roundrect (at 0.9125 0 270) (size 1.025 1.4) (layers F.Cu F.Paste F.Mask) (roundrect_rratio 0.243902)
+    (pad 2 smd roundrect (at 0.9125 0 270) (size 1.025 1.4) (layers F.Cu F.Paste F.Mask) (roundrect_rratio 0.2439014634146341)
       (net 1 GND))
-    (pad 1 smd roundrect (at -0.9125 0 270) (size 1.025 1.4) (layers F.Cu F.Paste F.Mask) (roundrect_rratio 0.243902)
+    (pad 1 smd roundrect (at -0.9125 0 270) (size 1.025 1.4) (layers F.Cu F.Paste F.Mask) (roundrect_rratio 0.2439014634146341)
       (net 23 /JuliaLCD/LED-))
     (model ${KISYS3DMOD}/Resistor_SMD.3dshapes/R_0805_2012Metric.wrl
@@
     (fp_line (start 1.7 -0.88) (end 1.7 0.88) (layer F.CrtYd) (width 0.05))
     (fp_line (start 1.7 0.88) (end -1.7 0.88) (layer F.CrtYd) (width 0.05))
-    (pad 2 smd roundrect (at 0.8875 0 90) (size 1.125 1.05) (layers F.Cu F.Paste F.Mask) (roundrect_rratio 0.238095)
+    (pad 2 smd roundrect (at 0.8875 0 90) (size 1.125 1.05) (layers F.Cu F.Paste F.Mask) (roundrect_rratio 0.2380942857142857)
       (net 1 GND))
-    (pad 1 smd roundrect (at -0.8875 0 90) (size 1.125 1.05) (layers F.Cu F.Paste F.Mask) (roundrect_rratio 0.238095)
+    (pad 1 smd roundrect (at -0.8875 0 90) (size 1.125 1.05) (layers F.Cu F.Paste F.Mask) (roundrect_rratio 0.2380942857142857)
       (net 8 "Net-(C46-Pad1)"))
     (model ${KISYS3DMOD}/Capacitor_Tantalum_SMD.3dshapes/CP_EIA-2012-15_AVX-P.wrl
@@
     (fp_line (start 1.7 0.88) (end 1.7 -0.88) (layer B.CrtYd) (width 0.05))
     (fp_line (start 1.7 -0.88) (end -1.7 -0.88) (layer B.CrtYd) (width 0.05))
-    (pad 2 smd roundrect (at 0.8875 0) (size 1.125 1.05) (layers B.Cu B.Paste B.Mask) (roundrect_rratio 0.238095)
+    (pad 2 smd roundrect (at 0.8875 0) (size 1.125 1.05) (layers B.Cu B.Paste B.Mask) (roundrect_rratio 0.2380942857142857)
       (net 1 GND))
-    (pad 1 smd roundrect (at -0.8875 0) (size 1.125 1.05) (layers B.Cu B.Paste B.Mask) (roundrect_rratio 0.238095)
+    (pad 1 smd roundrect (at -0.8875 0) (size 1.125 1.05) (layers B.Cu B.Paste B.Mask) (roundrect_rratio 0.2380942857142857)
       (net 4 +1V2))
     (model ${KISYS3DMOD}/Capacitor_Tantalum_SMD.3dshapes/CP_EIA-2012-15_AVX-P.wrl
@@
     (fp_line (start 1.7 0.88) (end 1.7 -0.88) (layer B.CrtYd) (width 0.05))
     (fp_line (start 1.7 -0.88) (end -1.7 -0.88) (layer B.CrtYd) (width 0.05))
-    (pad 2 smd roundrect (at 0.8875 0 180) (size 1.125 1.05) (layers B.Cu B.Paste B.Mask) (roundrect_rratio 0.238095)
+    (pad 2 smd roundrect (at 0.8875 0 180) (size 1.125 1.05) (layers B.Cu B.Paste B.Mask) (roundrect_rratio 0.2380942857142857)
       (net 1 GND))
-    (pad 1 smd roundrect (at -0.8875 0 180) (size 1.125 1.05) (layers B.Cu B.Paste B.Mask) (roundrect_rratio 0.238095)
+    (pad 1 smd roundrect (at -0.8875 0 180) (size 1.125 1.05) (layers B.Cu B.Paste B.Mask) (roundrect_rratio 0.2380942857142857)
       (net 2 +3V3))
     (model ${KISYS3DMOD}/Capacitor_Tantalum_SMD.3dshapes/CP_EIA-2012-15_AVX-P.wrl
@@
     )
   )
+  (gr_line (start 138.9 132.8) (end 78.4 132.8) (layer Edge.Cuts) (width 0.05))
+  (gr_line (start 138.9 86.8) (end 138.9 132.8) (layer Edge.Cuts) (width 0.05))
+  (gr_line (start 78.4 86.8) (end 138.9 86.8) (layer Edge.Cuts) (width 0.05))
+  (gr_line (start 78.4 132.8) (end 78.4 86.8) (layer Edge.Cuts) (width 0.05))
+  (gr_text "iank@iank.org\nv2.1.0.0" (at 81.4 130.6) (layer F.SilkS)
+    (effects (font (size 0.8 0.8) (thickness 0.1)) (justify left))
+  )
   (via (at 94.9 106.9) (size 0.45) (drill 0.2) (layers F.Cu B.Cu) (net 1))
