File: cad/v2.1_breakout/v2.1_breakout/v2.1_breakout.kicad_pcb (KiCad board)
At the start: 2 copper layers, 38.3 x 27.4 mm, 14 parts, among them J1 Altera Byte Blaster, J2 Julia v2.1.0.0 connector, J3 SiLabs USB Debug Header, J4 UART

Commit message: v2.1.1
Parts:
- J2: value Julia v2.1.0.0 connector -> Julia v2.1.1.0 connector; footprint ik:Hirose_DF23_DF23C-10DS-0.5V_2x05_P0.50mm_Vertical -> Connector_PinHeader_1.27mm:PinHeader_2x05_P1.27mm_Vertical
- moved J2 2.61 mm to (75.2, 166.0), turned to 0 degrees
Routing:
- net /TMS: track 50.8 -> 45.8 mm, vias 1 -> 2
- net /TDI: track 58.3 -> 53.7 mm, vias 1 -> 2
- net /UART0_TX: track 22.0 -> 25.7 mm, vias 2 -> 1
- net /UART0_RX: track 24.3 -> 27.6 mm, vias 2 -> 1
- net /TCK: track 36.3 -> 39.5 mm, vias 2 -> 1
- net /TDO: track 39.6 -> 42.8 mm, vias 2 -> 1
- net /C2D: track 47.0 -> 48.8 mm
- net /C2CK: track 34.7 -> 36.4 mm
- net /+3V3: track 36.4 -> 35.0 mm
- net /GND: vias 18 -> 17
