File: cad/v2.1_breakout/v2.1_breakout/v2.1_breakout.sch (KiCad schematic (older format))
At the start: 14 parts, among them J1 Altera Byte Blaster, J2 Julia v2.1.0.0 connector, J3 SiLabs USB Debug Header, J4 UART

Commit message: v2.1.1
Parts:
- J2: value Julia v2.1.0.0 connector -> Julia v2.1.1.0 connector; footprint ik:Hirose_DF23_DF23C-10DS-0.5V_2x05_P0.50mm_Vertical -> Connector_PinHeader_1.27mm:PinHeader_2x05_P1.27mm_Vertical
Changed lines of the file:
@@
 P 2800 2800
 F 0 "J2" H 2850 3217 50  0000 C CNN
-F 1 "Julia v2.1.0.0 connector" H 2850 3126 50  0000 C CNN
-F 2 "ik:Hirose_DF23_DF23C-10DS-0.5V_2x05_P0.50mm_Vertical" H 2800 2800 50  0001 C CNN
+F 1 "Julia v2.1.1.0 connector" H 2850 3126 50  0000 C CNN
+F 2 "Connector_PinHeader_1.27mm:PinHeader_2x05_P1.27mm_Vertical" H 2800 2800 50  0001 C CNN
 F 3 "~" H 2800 2800 50  0001 C CNN
 	1    2800 2800
