File: cad/v2.1.1.0/julia_v2.1.1.0/julia_config.sch (KiCad schematic (older format))
At the start: 8 parts, among them U5 W25Q80DVSNIG, U6 EFM8BB21F16I-C-QFN20

Commit message: Several more 3d models
Parts:
- U6: footprint Package_DFN_QFN:SiliconLabs_QFN-20-1EP_3x3mm_P0.5mm_EP1.8x1.8mm -> ik:SiliconLabs_QFN-20-1EP_3x3mm_P0.5mm_EP1.8x1.8mm
Changed lines of the file:
@@
 F 0 "U6" H 4300 3331 50  0000 C CNN
 F 1 "EFM8BB21F16I-C-QFN20" H 4300 3240 50  0000 C CNN
-F 2 "Package_DFN_QFN:SiliconLabs_QFN-20-1EP_3x3mm_P0.5mm_EP1.8x1.8mm" H 4300 3250 50  0001 C CNN
+F 2 "ik:SiliconLabs_QFN-20-1EP_3x3mm_P0.5mm_EP1.8x1.8mm" H 4300 3250 50  0001 C CNN
 F 3 "https://www.silabs.com/documents/public/data-sheets/efm8bb1-datasheet.pdf" H 4300 2450 50  0001 C CNN
 	1    4300 2450
